File: hardware/kicad/main/sensors.kicad_sch (KiCad schematic)
At the start: 17 parts, among them U30 TMAG5273A2QDBVR, U31 LIS2DW12TR

Commit message: Apply schematic review fixes; base board routes to 100% with zero DRC errors
- OLED VCC input disconnect is now a TPS22917 load switch (CT to VIN) instead
  of an AO3401A/2N7002 with no real inrush control
- TPD4E05U06 TVS on the TMAG5273 lines (floating 316L ring passes 2.4 mm away)
- piezo: 470R series + 1M bleed; LED_DIN pull-down moved to the shifter input
- base: explicit 2x4 DSBGA fan-out for the BQ25180, 0.4 mm power tracks,
  BAT+/GND silkscreen at the battery connector, JEITA NTC over the pack
- SPEC: side-entry link headers on both boards, 28 AWG power leads

Co-Authored-By: Claude Opus 5.5 <noreply@anthropic.com>
Claude-Session: https://claude.ai/code/session_01P3cqdBhxLcWY3sGUVf9LAJ
Parts:
- added R59: 1M, Resistor_SMD:R_0402_1005Metric, symbol Device:R
- added U32: TPD4E05U06DQAR, Package_SON:USON-10_2.5x1.0mm_P0.5mm, symbol Power_Protection:TPD4E05U06DQA
- R57, R58: value 100 -> 470; LCSC C25076 -> C25117; MPN 0402WGF1000TCE -> 0402WGF4700TCE
Connections:
- net BZ_N: now also R59.2
- net BZ_P: now also R59.1
- net GND: now also U32.3 (GND), U32.8 (GND)
- net TMAG_INT_N: now also U32.4 (D2+)
- net TMAG_SCL: now also U32.1 (D1+)
- net TMAG_SDA: now also U32.2 (D1-)
- no-connect marks 1 -> 6
Other:
- note added: "Encoder ESD (floating 316L ring 2.4 mm below)"
- note added: "The flywheel is a touchable, electrically floating metal ring passing under U30. U32 clamps TMAG_SCL/SDA/INT_N right at U30 (short GND return via next to U30)."
- moved on the sheet: BZ1, R50, R51, R52
